Commit message: add collision/inertial tags, add xacro file

File: src/robot_description/urdf/robot1.urdf (robot description, URDF)
Before this commit: robot robot1, 4 links, 3 joints
Links:
- added link wheel_4, mass 10; collision cylinder length=0.05 radius=0.05; visual cylinder length=0.05 radius=0.05
- link base_link: mass None -> 100; geometry collision box size=0.2 .3 0.1; visual box size=0.2 .3 .1
- link wheel_1: mass None -> 10; geometry collision cylinder length=0.05 radius=0.05; visual cylinder length=0.05 radius=0.05
- link wheel_2: mass None -> 10; geometry collision cylinder length=0.05 radius=0.05; visual cylinder length=0.05 radius=0.05
- link wheel_3: mass None -> 10; geometry collision cylinder length=0.05 radius=0.05; visual cylinder length=0.05 radius=0.05
Joints:
- added joint base_to_wheel4: type fixed, parent base_link, child wheel_4, origin xyz=0 0 0
